Commit message: Save progress

File: notebooks/four_wheel_robot.urdf (robot description, URDF)
Before this commit: robot four_wheel_robot, 5 links, 4 joints
Links:
- link left_front_wheel: geometry collision cylinder length=1.0 radius=1.0; visual cylinder length=1.0 radius=1.0
- link left_rear_wheel: geometry collision cylinder length=1.0 radius=1.0; visual cylinder length=1.0 radius=1.0
- link right_front_wheel: geometry collision cylinder length=1.0 radius=1.0; visual cylinder length=1.0 radius=1.0
- link right_rear_wheel: geometry collision cylinder length=1.0 radius=1.0; visual cylinder length=1.0 radius=1.0
Joints:
- joint left_front_wheel_joint: origin xyz=0.0 0.0 0.0 rpy=0.0 -0.0 0.0 -> xyz=0.25 0.25 0.0 rpy=0.0 0.0 0.0
- joint right_front_wheel_joint: origin xyz=0.0 0.0 0.0 rpy=0.0 -0.0 0.0 -> xyz=1.0 0.25 0.0 rpy=0.0 0.0 0.0
