Commit message: Fix error in meshing to visualize Via URDF

File: notebooks/Axle column test_scaled.urdf (robot description, URDF)
Before this commit: robot Axle column test, 2 links, 1 joints
Links:
- link LEFT_FRONT_axle: geometry collision cylinder length=3.5000000000000004 radius=0.166; visual cylinder length=3.5000000000000004 radius=0.166
- link LEFT_FRONT_steering_column: geometry collision cylinder length=4.83 radius=0.2; visual cylinder length=4.83 radius=0.2
Joints:
- joint LEFT_FRONT_axle_to_LEFT_FRONT_steering_column_joint: origin xyz=0.0483 0.0 0.0 rpy=0.0 1.5707963267948966 0.0 -> xyz=0.48300000000000004 0.0 0.0 rpy=0.0 1.5707963267948966 0.0
