Commit message: Reorganize properties

File: notebooks/wheel_axle_test.urdf (robot description, URDF)
Before this commit: robot wheel_axle_test, 2 links, 1 joints
Joints:
- joint LEFT_FRONT_to_LEFT_FRONT_axle_joint: origin xyz=0.0 0.0 0.0 rpy=0.0 0.0 0.0 -> xyz=0.0 0.0 0.004500000000000001 rpy=0.0 0.0 0.0
